Commit message: Modify urdf

File: src/wd_description/src/gazebo_control.xacro (robot description, xacro)
@@ -4,10 +4,10 @@
         <plugin name="gz::sim::systems::DiffDrive" filename="gz-sim-diff-drive-system">
             <!-- Wheel Information -->
-            <left_joint>left_wheel_joint</left_joint>
-            <right_joint>right_wheel_joint</right_joint>
-            <wheel_separation>0.35</wheel_separation>
-            <wheel_radius>0.05</wheel_radius>
+            <left_joint>wheel_left_joint</left_joint>
+            <right_joint>wheel_right_joint</right_joint>
+            <wheel_separation>0.196</wheel_separation>
+            <wheel_radius>0.0325</wheel_radius>
             <!-- Input -->
-            <topic>cmd_vel</topic>
+            <topic>/cmd_vel</topic>
             <!-- Output -->
             <frame_id>odom</frame_id>
@@ -18,6 +18,6 @@
         <plugin name="gz::sim::systems::JointStatePublisher" filename="gz-sim-joint-state-publisher-system">
             <topic>joint_states</topic>
-            <joint_name>left_wheel_joint</joint_name>
-            <joint_name>right_wheel_joint</joint_name>
+            <joint_name>wheel_left_joint</joint_name>
+            <joint_name>wheel_right_joint</joint_name>
         </plugin>
     </gazebo>

File: src/wd_description/src/robot.urdf.xacro (robot description, xacro)
@@ -1,5 +1,5 @@
 <?xml version="1.0"?>
 <robot xmlns:xacro="http://www.ros.org/wiki/xacro"  name="robot">
-    <xacro:include filename="robot_core.xacro" />
+    <xacro:include filename="robot_desc.xacro" />
     <xacro:include filename="gazebo_control.xacro"/>
 </robot>

File: src/wd_description/src/robot_desc.xacro (robot description, xacro)
@@ -39,7 +39,12 @@
         </geometry>
         </collision>
-        <xacro:inertial_box mass="m" x="x" y="y" z="z">
-            <origin xyz="" rpy="0 0 0"/>
-        </xacro:inertial_box>
+        <inertial>
+            <origin xyz="0.097 0.003 0.029" rpy="0 0 0"/>
+            <mass value="1.227"/>
+            <inertia
+            ixx="3.86E-03" ixy="0" ixz="0"
+            iyy="6.37E-03" iyz="0"
+            izz="8.57E-03"/>
+        </inertial>
     </link>
     <joint name="chassis_joint" type="fixed">
@@ -61,7 +66,12 @@
         </geometry>
         </collision>
-        <xacro:inertial_box mass="m" x="x" y="y" z="z">
-            <origin xyz="" rpy="0 0 0"/>
-        </xacro:inertial_box>
+        <inertial>
+            <origin xyz="0 0 0.005" rpy="0 0 0"/>
+            <mass value="0.182"/>
+            <inertia
+            ixx="1.79E-04" ixy="0" ixz="0"
+            iyy="1.43E-04" iyz="0"
+            izz="2.85E-04"/>
+        </inertial>
     </link>
     <joint name="jetson_joint" type="fixed">
@@ -76,5 +86,5 @@
             <mesh filename="file:///home/logicbomb/Projects/SLAM/wheely-dan/src/wd_description/meshes/battery_link.stl" scale="0.001 0.001 0.001"/>
         </geometry>
-        </material name="red"/>
+        <material name="red"/>
         </visual>
         <collision>
@@ -83,7 +93,12 @@
         </geometry>
         </collision>
-        <xacro:inertial_box mass="m" x="x" y="y" z="z">
-            <origin xyz="" rpy="0 0 0"/>
-        </xacro:inertial_box>
+        <inertial>
+            <origin xyz="0 0 0.0115" rpy="0 0 0"/>
+            <mass value="0.178"/>
+            <inertia
+            ixx="1.71E-04" ixy="0" ixz="0"
+            iyy="2.50E-05" iyz="0"
+            izz="1.81E-04"/>
+        </inertial>
     </link>
     <joint name="battery_joint" type="fixed">
@@ -105,7 +120,12 @@
         </geometry>
         </collision>
-        <xacro:inertial_box mass="m" x="x" y="y" z="z">
-            <origin xyz="" rpy="0 0 0"/>
-        </xacro:inertial_box>
+        <inertial>
+            <origin xyz="0 0 0" rpy="0 0 0"/>
+            <mass value="0.04"/>
+            <inertia
+            ixx="2.41E-05" ixy="0" ixz="0"
+            iyy="2.13E-05" iyz="0"
+            izz="4.54E-05"/>
+        </inertial>
     </link>
     <joint name="pcb_joint" type="fixed">
@@ -127,7 +147,12 @@
         </geometry>
         </collision>
-        <xacro:inertial_box mass="m" x="x" y="y" z="z">
-            <origin xyz="" rpy="0 0 0"/>
-        </xacro:inertial_box>
+        <inertial>
+            <origin xyz="0 0 0" rpy="0 0 0"/>
+            <mass value="0.02"/>
+            <inertia
+            ixx="6.24E-06" ixy="0" ixz="0"
+            iyy="1.86E-06" iyz="0"
+            izz="8.02E-06"/>
+        </inertial>
     </link>
     <joint name="driver_left_joint" type="fixed">
@@ -149,7 +174,12 @@
         </geometry>
         </collision>
-        <xacro:inertial_box mass="m" x="x" y="y" z="z">
-            <origin xyz="" rpy="0 0 0"/>
-        </xacro:inertial_box>
+        <inertial>
+            <origin xyz="0 0 0" rpy="0 0 0"/>
+            <mass value="0.02"/>
+            <inertia
+            ixx="6.24E-06" ixy="0" ixz="0"
+            iyy="1.86E-06" iyz="0"
+            izz="8.02E-06"/>
+        </inertial>
     </link>
     <joint name="driver_right_joint" type="fixed">
@@ -158,4 +188,32 @@
         <origin xyz="0.04576 -0.03548 0.018"/>
     </joint>
+    <!-- ========= LIDAR ========= -->
+    <link name="lidar_link">
+        <visual>
+        <geometry>
+            <mesh filename="file:///home/logicbomb/Projects/SLAM/wheely-dan/src/wd_description/meshes/lidar_link.stl" scale="0.001 0.001 0.001"/>
+        </geometry>
+        <material name="white"/>
+        </visual>
+        <collision>
+        <geometry>
+            <mesh filename="file:///home/logicbomb/Projects/SLAM/wheely-dan/src/wd_description/meshes/lidar_link.stl" scale="0.001 0.001 0.001"/>
+        </geometry>
+        </collision>
+        <!-- done -->
+        <inertial>
+            <origin xyz="0 0 0.0275" rpy="0 0 0"/>
+            <mass value="0.187"/>
+            <inertia
+            ixx="1.23E-04" ixy="0" ixz="0"
+            iyy="2.03E-04" iyz="0"
+            izz="2.32E-04"/>
+        </inertial>
+    </link>
+    <joint name="lidar_joint" type="fixed">
+        <parent link="base_link"/>
+        <child link="lidar_link"/>
+        <origin xyz="0.006175 0 0.095"/>
+    </joint>
     <!-- ========= WHEEL L ========= -->
     <link name="wheel_left_link">
@@ -171,7 +229,12 @@
         </geometry>
         </collision>
-        <xacro:inertial_cylinder mass="0.1" length="0.04" radius="0.05">
-            <origin xyz="0 0 0" rpy="0 0 0"/>
-        </xacro:inertial_cylinder>
+        <inertial>
+            <origin xyz="0 0.003 0" rpy="0 0 0"/>
+            <mass value="0.046"/>
+            <inertia
+            ixx="1.45E-05" ixy="0" ixz="0"
+            iyy="2.43E-05" iyz="0"
+            izz="1.45E-05"/>
+        </inertial>
     </link>
     <joint name="wheel_left_joint" type="continuous">
@@ -194,7 +257,12 @@
         </geometry>
         </collision>
-        <xacro:inertial_cylinder mass="0.1" length="0.04" radius="0.05">
-            <origin xyz="0 0 0" rpy="0 0 0"/>
-        </xacro:inertial_cylinder>
+        <inertial>
+            <origin xyz="0 -0.003 0" rpy="0 0 0"/>
+            <mass value="0.046"/>
+            <inertia
+            ixx="1.45E-05" ixy="0" ixz="0"
+            iyy="2.43E-05" iyz="0"
+            izz="1.45E-05"/>
+        </inertial>
     </link>
     <joint name="wheel_right_joint" type="continuous">
@@ -217,7 +285,12 @@
         </geometry>
         </collision>
-        <xacro:inertial_cylinder mass="0.1" length="0.04" radius="0.05">
-            <origin xyz="0 0 0" rpy="0 0 0"/>
-        </xacro:inertial_cylinder>
+        <inertial>
+            <origin xyz="0 0 -0.004" rpy="0 0 0"/>
+            <mass value="0.01"/>
+            <inertia
+            ixx="2.79E-07" ixy="0" ixz="0"
+            iyy="2.79E-07" iyz="0"
+            izz="4.51E-07"/>
+        </inertial>
     </link>
     <joint name="caster_fork_left_joint" type="fixed">
@@ -238,7 +311,12 @@
         </geometry>
         </collision>
-        <xacro:inertial_cylinder mass="0.1" length="0.04" radius="0.05">
-            <origin xyz="0 0 0" rpy="0 0 0"/>
-        </xacro:inertial_cylinder>
+        <inertial>
+            <origin xyz="0 0 0" rpy="0 0 0"/>
+            <mass value="0.004"/>
+            <inertia
+            ixx="6.30E-08" ixy="0" ixz="0"
+            iyy="7.20E-08" iyz="0"
+            izz="6.30E-08"/>
+        </inertial>
     </link>
     <joint name="caster_wheel_left_joint" type="continuous">
@@ -261,7 +339,12 @@
         </geometry>
         </collision>
-        <xacro:inertial_cylinder mass="0.1" length="0.04" radius="0.05">
-            <origin xyz="0 0 0" rpy="0 0 0"/>
-        </xacro:inertial_cylinder>
+        <inertial>
+            <origin xyz="0 0 -0.004" rpy="0 0 0"/>
+            <mass value="0.01"/>
+            <inertia
+            ixx="2.79E-07" ixy="0" ixz="0"
+            iyy="2.79E-07" iyz="0"
+            izz="4.51E-07"/>
+        </inertial>
     </link>
     <joint name="caster_fork_right_joint" type="fixed">
@@ -282,7 +365,12 @@
         </geometry>
         </collision>
-        <xacro:inertial_cylinder mass="0.1" length="0.04" radius="0.05">
-            <origin xyz="0 0 0" rpy="0 0 0"/>
-        </xacro:inertial_cylinder>
+        <inertial>
+            <origin xyz="0 0 0" rpy="0 0 0"/>
+            <mass value="0.004"/>
+            <inertia
+            ixx="6.30E-08" ixy="0" ixz="0"
+            iyy="7.20E-08" iyz="0"
+            izz="6.30E-08"/>
+        </inertial>
     </link>
     <joint name="caster_wheel_right_joint" type="continuous">
@@ -292,26 +380,3 @@
         <axis xyz="0 1 0"/>
     </joint>
-    <!-- ========= LIDAR ========= -->
-    <link name="lidar_link">
-        <visual>
-        <geometry>
-            <mesh filename="file:///home/logicbomb/Projects/SLAM/wheely-dan/src/wd_description/meshes/lidar_link.stl" scale="0.001 0.001 0.001"/>
-        </geometry>
-        <material name="white"/>
-        </visual>
-        <collision>
-        <geometry>
-            <mesh filename="file:///home/logicbomb/Projects/SLAM/wheely-dan/src/wd_description/meshes/lidar_link.stl" scale="0.001 0.001 0.001"/>
-        </geometry>
-        </collision>
-        <!-- done -->
-        <xacro:inertial_box mass="0.187" x="0.1" y="0.07" z="0.055">
-            <origin xyz="0 0 0.0275" rpy="0 0 0"/>
-        </xacro:inertial_box>
-    </link>
-    <joint name="lidar_joint" type="fixed">
-        <parent link="base_link"/>
-        <child link="lidar_link"/>
-        <origin xyz="0.006175 0 0.095"/>
-    </joint>
 </robot>

Commit message: Change torque limit and change Twist type

File: src/wd_description/src/gazebo_control.xacro (robot description, xacro)
@@ -9,5 +9,5 @@
             <wheel_radius>0.0325</wheel_radius>
             <!-- Input -->
-            <topic>/cmd_vel</topic>
+            <topic>cmd_vel</topic>
             <!-- Output -->
             <frame_id>odom</frame_id>

File: src/wd_description/src/robot_desc.xacro (robot description, xacro)
@@ -225,5 +225,5 @@
         <collision>
         <geometry>
-            <mesh filename="file:///home/logicbomb/Projects/SLAM/wheely-dan/src/wd_description/meshes/wheel_left_link.stl" scale="0.001 0.001 0.001"/>
+            <sphere radius="0.0325"/>
         </geometry>
         </collision>
@@ -242,5 +242,5 @@
         <origin xyz="0 0.098 0.0145"/>
         <axis xyz="0 1 0"/>
-        <limit effort="0.05" velocity="10.0"/>
+        <limit effort="100.0" velocity="1000.0"/>
     </joint>
     <!-- ========= WHEEL R ========= -->
@@ -254,5 +254,5 @@
         <collision>
         <geometry>
-            <mesh filename="file:///home/logicbomb/Projects/SLAM/wheely-dan/src/wd_description/meshes/wheel_right_link.stl" scale="0.001 0.001 0.001"/>
+            <sphere radius="0.0325"/>
         </geometry>
         </collision>
@@ -271,5 +271,5 @@
         <origin xyz="0 -0.098 0.0145"/>
         <axis xyz="0 1 0"/>
-        <limit effort="0.05" velocity="10.0"/>
+        <limit effort="100.0" velocity="1000.0"/>
     </joint>
     <!-- ========= CASTER L ========= -->

Commit message: Update urdf files for new motor positions

File: src/wd_description/src/gazebo_control.xacro (robot description, xacro)
@@ -6,5 +6,5 @@
             <left_joint>wheel_left_joint</left_joint>
             <right_joint>wheel_right_joint</right_joint>
-            <wheel_separation>0.196</wheel_separation>
+            <wheel_separation>0.202</wheel_separation>
             <wheel_radius>0.0325</wheel_radius>
             <!-- Input -->

File: src/wd_description/src/robot_desc.xacro (robot description, xacro)
@@ -196,5 +196,4 @@
         </geometry>
         </collision>
-        <!-- done -->
         <inertial>
             <origin xyz="0 0 0.0275" rpy="0 0 0"/>
@@ -220,4 +219,5 @@
         </visual>
         <collision>
+        <origin xyz="0 0.003 0" rpy="0 0 0"/>
         <geometry>
             <sphere radius="0.0325"/>
@@ -236,5 +236,5 @@
         <parent link="base_link"/>
         <child link="wheel_left_link"/>
-        <origin xyz="0 0.098 0.0145"/>
+        <origin xyz="0 0.099 0.0125"/>
         <axis xyz="0 1 0"/>
     </joint>
@@ -248,4 +248,5 @@
         </visual>
         <collision>
+        <origin xyz="0 -0.003 0" rpy="0 0 0"/>
         <geometry>
             <sphere radius="0.0325"/>
@@ -264,5 +265,5 @@
         <parent link="base_link"/>
         <child link="wheel_right_link"/>
-        <origin xyz="0 -0.098 0.0145"/>
+        <origin xyz="0 -0.099 0.0125"/>
         <axis xyz="0 1 0"/>
     </joint>
