Commit message: WIP gz depth camera

File: src/wd_description/src/robot.urdf.xacro (robot description, xacro)
@@ -11,3 +11,4 @@
     </xacro:unless>
     <xacro:include filename="$(find wd_simulation)/urdf/gazebo_lidar.xacro"/>
+    <xacro:include filename="$(find wd_simulation)/urdf/gazebo_depth_camera.xacro"/>
 </robot>

File: src/wd_description/src/robot_desc.xacro (robot description, xacro)
@@ -375,4 +375,29 @@
         <origin xyz="-0.01 0 -0.0107"/>
         <axis xyz="0 1 0"/>
+    </joint>
+    <!-- ========= DEPTH CAMERA ========= -->
+    <link name="depth_camera_link">
+        <visual>
+        <geometry>
+            <box size="0.3 0.3 0.15"/>
+        </geometry>
+        <material name="dark_grey"/>
+        </visual>
+        <collision>
+        <geometry>
+            <box size="0.3 0.3 0.15"/>
+        </geometry>
+        </collision>
+        <inertial>
+            <mass value="0.072"/>
+            <inertia ixx="0.000004" ixy="0" ixz="0"
+                    iyy="0.000024" iyz="0"
+                    izz="0.000025"/>
+        </inertial>
+    </link>
+    <joint name="depth_camera_joint" type="fixed">
+        <parent link="base_link"/>
+        <child link="depth_camera_link"/>
+        <origin xyz="0.056175 0 0.095"/>
     </joint>
     <!-- ========= GAZEBO SETTINGS ========= -->

Commit message: WIP 3d mapping

File: src/wd_description/src/robot.urdf.xacro (robot description, xacro)
@@ -10,5 +10,4 @@
         <xacro:include filename="$(find wd_simulation)/urdf/gazebo_control.xacro"/>
     </xacro:unless>
-    <xacro:include filename="$(find wd_simulation)/urdf/gazebo_lidar.xacro"/>
-    <xacro:include filename="$(find wd_simulation)/urdf/gazebo_depth_camera.xacro"/>
+    <xacro:include filename="$(find wd_simulation)/urdf/sensors.xacro"/>
 </robot>

File: src/wd_description/src/robot_desc.xacro (robot description, xacro)
@@ -380,11 +380,11 @@
         <visual>
         <geometry>
-            <box size="0.3 0.3 0.15"/>
-        </geometry>
-        <material name="dark_grey"/>
-        </visual>
-        <collision>
-        <geometry>
-            <box size="0.3 0.3 0.15"/>
+            <box size="0.003 0.003 0.0015"/>
+        </geometry>
+        <material name="dark_grey"/>
+        </visual>
+        <collision>
+        <geometry>
+            <box size="0.003 0.003 0.0015"/>
         </geometry>
         </collision>
@@ -399,6 +399,14 @@
         <parent link="base_link"/>
         <child link="depth_camera_link"/>
-        <origin xyz="0.056175 0 0.095"/>
-    </joint>
+        <origin xyz="0.1 0 0.2"/>
+    </joint>
+    <!-- ── Optical frame (ROS convention: z-forward, x-right, y-down) ── -->
+    <joint name="depth_camera_optical_joint" type="fixed">
+      <parent link="depth_camera_link"/>
+      <child  link="depth_camera_optical_frame"/>
+      <!-- Rotate from Gazebo (x-forward) to ROS optical (z-forward) convention -->
+      <origin xyz="0 0 0" rpy="${-pi/2} 0 ${-pi/2}"/>
+    </joint>
+    <link name="depth_camera_optical_frame"/>
     <!-- ========= GAZEBO SETTINGS ========= -->
     <gazebo reference="caster_wheel_left_link">
