Commit message: Modify launch files

File: src/wd_description/src/robot_desc.xacro (robot description, xacro)
@@ -1,10 +1,9 @@
 <?xml version="1.0"?>
 <robot name="wheely_dan" xmlns:xacro="http://www.ros.org/wiki/xacro">
-    <xacro:include filename="inertial_macros.xacro" />
     <material name="white">
         <color rgba="1 1 1 1"/>
     </material>
     <material name="red">
-        <color rgba="1 0 0 1"/>
+        <color rgba="0.3 0 0 1"/>
     </material>
     <material name="orange">
@@ -12,14 +11,14 @@
     </material>
     <material name="blue">
-        <color rgba="0.2 0.2 1 1"/>
-    </material>
-    <material name="black">
-        <color rgba="0 0 0 1"/>
+        <color rgba="0 0 0.05 1"/>
     </material>
     <material name="grey">
-        <color rgba="0.5 0.5 0.5 1"/>
+        <color rgba="0.4 0.4 0.4 1"/>
+    </material>
+    <material name="dark_grey">
+        <color rgba="0.2 0.2 0.2 1"/>
     </material>
     <material name="green">
-        <color rgba="0 1 0 1"/>
+        <color rgba="0.125 0.3 0 1"/>
     </material>
     <!-- ========= BASE ========= -->
@@ -32,5 +31,5 @@
             <mesh filename="file:///home/logicbomb/Projects/SLAM/wheely-dan/src/wd_description/meshes/chassis_link.stl" scale="0.001 0.001 0.001"/>
         </geometry>
-        <material name="black"/>
+        <material name="grey"/>
         </visual>
         <collision>
@@ -59,5 +58,5 @@
             <mesh filename="file:///home/logicbomb/Projects/SLAM/wheely-dan/src/wd_description/meshes/jetson_link.stl" scale="0.001 0.001 0.001"/>
         </geometry>
-        <material name="grey"/>
+        <material name="dark_grey"/>
         </visual>
         <collision>
@@ -140,5 +139,5 @@
             <mesh filename="file:///home/logicbomb/Projects/SLAM/wheely-dan/src/wd_description/meshes/driver_left_link.stl" scale="0.001 0.001 0.001"/>
         </geometry>
-        <material name="black"/>
+        <material name="grey"/>
         </visual>
         <collision>
@@ -167,5 +166,5 @@
             <mesh filename="file:///home/logicbomb/Projects/SLAM/wheely-dan/src/wd_description/meshes/driver_right_link.stl" scale="0.001 0.001 0.001"/>
         </geometry>
-        <material name="black"/>
+        <material name="grey"/>
         </visual>
         <collision>
@@ -194,5 +193,5 @@
             <mesh filename="file:///home/logicbomb/Projects/SLAM/wheely-dan/src/wd_description/meshes/lidar_link.stl" scale="0.001 0.001 0.001"/>
         </geometry>
-        <material name="white"/>
+        <material name="dark_grey"/>
         </visual>
         <collision>
@@ -243,4 +242,5 @@
         <origin xyz="0 0.098 0.0145"/>
         <axis xyz="0 1 0"/>
+        <limit effort="0.05" velocity="10.0"/>
     </joint>
     <!-- ========= WHEEL R ========= -->
@@ -271,4 +271,5 @@
         <origin xyz="0 -0.098 0.0145"/>
         <axis xyz="0 1 0"/>
+        <limit effort="0.05" velocity="10.0"/>
     </joint>
     <!-- ========= CASTER L ========= -->
@@ -278,5 +279,5 @@
             <mesh filename="file:///home/logicbomb/Projects/SLAM/wheely-dan/src/wd_description/meshes/caster_fork_link.stl" scale="0.001 0.001 0.001"/>
         </geometry>
-        <material name="grey"/>
+        <material name="dark_grey"/>
         </visual>
         <collision>
@@ -304,5 +305,5 @@
             <mesh filename="file:///home/logicbomb/Projects/SLAM/wheely-dan/src/wd_description/meshes/caster_wheel_link.stl" scale="0.001 0.001 0.001"/>
         </geometry>
-        <material name="black"/>
+        <material name="dark_grey"/>
         </visual>
         <collision>
@@ -332,5 +333,5 @@
             <mesh filename="file:///home/logicbomb/Projects/SLAM/wheely-dan/src/wd_description/meshes/caster_fork_link.stl" scale="0.001 0.001 0.001"/>
         </geometry>
-        <material name="grey"/>
+        <material name="dark_grey"/>
         </visual>
         <collision>
@@ -358,5 +359,5 @@
             <mesh filename="file:///home/logicbomb/Projects/SLAM/wheely-dan/src/wd_description/meshes/caster_wheel_link.stl" scale="0.001 0.001 0.001"/>
         </geometry>
-        <material name="black"/>
+        <material name="dark_grey"/>
         </visual>
         <collision>
@@ -380,3 +381,12 @@
         <axis xyz="0 1 0"/>
     </joint>
+    <!-- ========= GAZEBO SETTINGS ========= -->
+    <gazebo reference="caster_wheel_left_link">
+        <mu1 value="0.0"/>
+        <mu2 value="0.0"/>
+    </gazebo>
+    <gazebo reference="caster_wheel_right_link">
+        <mu1 value="0.0"/>
+        <mu2 value="0.0"/>
+    </gazebo>
 </robot>

Commit message: Add depth camera in gz

File: src/wd_description/src/robot_desc.xacro (robot description, xacro)
@@ -379,12 +379,14 @@
     <link name="depth_camera_link">
         <visual>
-        <geometry>
-            <box size="0.003 0.003 0.0015"/>
-        </geometry>
-        <material name="dark_grey"/>
-        </visual>
-        <collision>
-        <geometry>
-            <box size="0.003 0.003 0.0015"/>
+        <origin xyz="0 0 0" rpy="${-pi/2} 0 ${-pi/2}"/>
+        <geometry>
+            <mesh filename="file:///home/logicbomb/Projects/SLAM/wheely-dan/src/wd_description/meshes/d435.dae"/>
+        </geometry>
+        <material name="dark_grey"/>
+        </visual>
+        <collision>
+        <origin xyz="0 0 0" rpy="${-pi/2} 0 ${-pi/2}"/>
+        <geometry>
+            <mesh filename="file:///home/logicbomb/Projects/SLAM/wheely-dan/src/wd_description/meshes/d435.dae"/>
         </geometry>
         </collision>
@@ -399,5 +401,5 @@
         <parent link="base_link"/>
         <child link="depth_camera_link"/>
-        <origin xyz="0.1 0 0.2"/>
+        <origin xyz="0.2 0 0.075" rpy="0 0 0"/>
     </joint>
     <!-- ── Optical frame (ROS convention: z-forward, x-right, y-down) ── -->

Commit message: Fix depth camera and add rtabmap

File: src/wd_description/src/robot_desc.xacro (robot description, xacro)
@@ -35,6 +35,7 @@
         </visual>
         <collision>
-        <geometry>
-            <mesh filename="file:///home/logicbomb/Projects/SLAM/wheely-dan/src/wd_description/meshes/chassis_link.stl" scale="0.001 0.001 0.001"/>
+        <origin xyz="0.1125 0 0.044" rpy="0 0 0"/>
+        <geometry>
+            <box size="0.225 0.17 0.088"/>
         </geometry>
         </collision>
@@ -56,9 +57,4 @@
         <material name="dark_grey"/>
         </visual>
-        <collision>
-        <geometry>
-            <mesh filename="file:///home/logicbomb/Projects/SLAM/wheely-dan/src/wd_description/meshes/jetson_link.stl" scale="0.001 0.001 0.001"/>
-        </geometry>
-        </collision>
         <inertial>
             <origin xyz="0 0 0.005" rpy="0 0 0"/>
@@ -83,9 +79,4 @@
         <material name="red"/>
         </visual>
-        <collision>
-        <geometry>
-            <mesh filename="file:///home/logicbomb/Projects/SLAM/wheely-dan/src/wd_description/meshes/battery_link.stl" scale="0.001 0.001 0.001"/>
-        </geometry>
-        </collision>
         <inertial>
             <origin xyz="0 0 0.0115" rpy="0 0 0"/>
@@ -110,9 +101,4 @@
         <material name="green"/>
         </visual>
-        <collision>
-        <geometry>
-            <mesh filename="file:///home/logicbomb/Projects/SLAM/wheely-dan/src/wd_description/meshes/pcb_link.stl" scale="0.001 0.001 0.001"/>
-        </geometry>
-        </collision>
         <inertial>
             <origin xyz="0 0 0" rpy="0 0 0"/>
@@ -137,9 +123,4 @@
         <material name="grey"/>
         </visual>
-        <collision>
-        <geometry>
-            <mesh filename="file:///home/logicbomb/Projects/SLAM/wheely-dan/src/wd_description/meshes/driver_left_link.stl" scale="0.001 0.001 0.001"/>
-        </geometry>
-        </collision>
         <inertial>
             <origin xyz="0 0 0" rpy="0 0 0"/>
@@ -164,9 +145,4 @@
         <material name="grey"/>
         </visual>
-        <collision>
-        <geometry>
-            <mesh filename="file:///home/logicbomb/Projects/SLAM/wheely-dan/src/wd_description/meshes/driver_right_link.stl" scale="0.001 0.001 0.001"/>
-        </geometry>
-        </collision>
         <inertial>
             <origin xyz="0 0 0" rpy="0 0 0"/>
@@ -191,9 +167,4 @@
         <material name="dark_grey"/>
         </visual>
-        <collision>
-        <geometry>
-            <mesh filename="file:///home/logicbomb/Projects/SLAM/wheely-dan/src/wd_description/meshes/lidar_link.stl" scale="0.001 0.001 0.001"/>
-        </geometry>
-        </collision>
         <inertial>
             <origin xyz="0 0 0.0275" rpy="0 0 0"/>
@@ -276,9 +247,4 @@
         <material name="dark_grey"/>
         </visual>
-        <collision>
-        <geometry>
-            <mesh filename="file:///home/logicbomb/Projects/SLAM/wheely-dan/src/wd_description/meshes/caster_fork_link.stl" scale="0.001 0.001 0.001"/>
-        </geometry>
-        </collision>
         <inertial>
             <origin xyz="0 0 -0.004" rpy="0 0 0"/>
@@ -330,9 +296,4 @@
         <material name="dark_grey"/>
         </visual>
-        <collision>
-        <geometry>
-            <mesh filename="file:///home/logicbomb/Projects/SLAM/wheely-dan/src/wd_description/meshes/caster_fork_link.stl" scale="0.001 0.001 0.001"/>
-        </geometry>
-        </collision>
         <inertial>
             <origin xyz="0 0 -0.004" rpy="0 0 0"/>
@@ -385,10 +346,4 @@
         <material name="dark_grey"/>
         </visual>
-        <collision>
-        <origin xyz="0 0 0" rpy="${-pi/2} 0 ${-pi/2}"/>
-        <geometry>
-            <mesh filename="file:///home/logicbomb/Projects/SLAM/wheely-dan/src/wd_description/meshes/d435.dae"/>
-        </geometry>
-        </collision>
         <inertial>
             <mass value="0.072"/>
@@ -406,9 +361,9 @@
     <joint name="depth_camera_optical_joint" type="fixed">
       <parent link="depth_camera_link"/>
-      <child  link="depth_camera_optical_frame"/>
+      <child  link="depth_camera_link_optical"/>
       <!-- Rotate from Gazebo (x-forward) to ROS optical (z-forward) convention -->
       <origin xyz="0 0 0" rpy="${-pi/2} 0 ${-pi/2}"/>
     </joint>
-    <link name="depth_camera_optical_frame"/>
+    <link name="depth_camera_link_optical"/>
     <!-- ========= GAZEBO SETTINGS ========= -->
     <gazebo reference="caster_wheel_left_link">

File: src/wd_simulation/urdf/sensors.xacro (robot description, xacro)
@@ -36,5 +36,5 @@
         <visualize>false</visualize>
         <always_on>1</always_on>
-        <update_rate>30</update_rate>
+        <update_rate>15</update_rate>
         <camera name="rs_front">
           <horizontal_fov>1.50098</horizontal_fov>
@@ -66,10 +66,10 @@
           <clip>
             <near>0.01</near>
-            <far>300</far>
+            <far>15</far>
           </clip>
           <depth_camera>
             <clip>
               <near>0.1</near>
-              <far>10</far>
+              <far>6</far>
             </clip>
           </depth_camera>
@@ -81,5 +81,5 @@
         </camera>
         <topic>camera/depth</topic>
-        <gz_frame_id>depth_camera_link</gz_frame_id>
+        <gz_frame_id>depth_camera_link_optical</gz_frame_id>
       </sensor>
     </gazebo>

Commit message: Change path names for modularity

File: src/wd_description/src/robot_desc.xacro (robot description, xacro)
@@ -30,5 +30,5 @@
         <visual>
         <geometry>
-            <mesh filename="file:///home/logicbomb/Projects/SLAM/wheely-dan/src/wd_description/meshes/chassis_link.stl" scale="0.001 0.001 0.001"/>
+            <mesh filename="$(find wd_description)/meshes/chassis_link.stl" scale="0.001 0.001 0.001"/>
         </geometry>
         <material name="grey"/>
@@ -53,5 +53,5 @@
         <visual>
         <geometry>
-            <mesh filename="file:///home/logicbomb/Projects/SLAM/wheely-dan/src/wd_description/meshes/jetson_link.stl" scale="0.001 0.001 0.001"/>
+            <mesh filename="$(find wd_description)/meshes/jetson_link.stl" scale="0.001 0.001 0.001"/>
         </geometry>
         <material name="dark_grey"/>
@@ -75,5 +75,5 @@
         <visual>
         <geometry>
-            <mesh filename="file:///home/logicbomb/Projects/SLAM/wheely-dan/src/wd_description/meshes/battery_link.stl" scale="0.001 0.001 0.001"/>
+            <mesh filename="$(find wd_description)/meshes/battery_link.stl" scale="0.001 0.001 0.001"/>
         </geometry>
         <material name="red"/>
@@ -97,5 +97,5 @@
         <visual>
         <geometry>
-            <mesh filename="file:///home/logicbomb/Projects/SLAM/wheely-dan/src/wd_description/meshes/pcb_link.stl" scale="0.001 0.001 0.001"/>
+            <mesh filename="$(find wd_description)/meshes/pcb_link.stl" scale="0.001 0.001 0.001"/>
         </geometry>
         <material name="green"/>
@@ -119,5 +119,5 @@
         <visual>
         <geometry>
-            <mesh filename="file:///home/logicbomb/Projects/SLAM/wheely-dan/src/wd_description/meshes/driver_left_link.stl" scale="0.001 0.001 0.001"/>
+            <mesh filename="$(find wd_description)/meshes/driver_left_link.stl" scale="0.001 0.001 0.001"/>
         </geometry>
         <material name="grey"/>
@@ -141,5 +141,5 @@
         <visual>
         <geometry>
-            <mesh filename="file:///home/logicbomb/Projects/SLAM/wheely-dan/src/wd_description/meshes/driver_right_link.stl" scale="0.001 0.001 0.001"/>
+            <mesh filename="$(find wd_description)/meshes/driver_right_link.stl" scale="0.001 0.001 0.001"/>
         </geometry>
         <material name="grey"/>
@@ -163,5 +163,5 @@
         <visual>
         <geometry>
-            <mesh filename="file:///home/logicbomb/Projects/SLAM/wheely-dan/src/wd_description/meshes/lidar_link.stl" scale="0.001 0.001 0.001"/>
+            <mesh filename="$(find wd_description)/meshes/lidar_link.stl" scale="0.001 0.001 0.001"/>
         </geometry>
         <material name="dark_grey"/>
@@ -185,5 +185,5 @@
         <visual>
         <geometry>
-            <mesh filename="file:///home/logicbomb/Projects/SLAM/wheely-dan/src/wd_description/meshes/wheel_left_link.stl" scale="0.001 0.001 0.001"/>
+            <mesh filename="$(find wd_description)/meshes/wheel_left_link.stl" scale="0.001 0.001 0.001"/>
         </geometry>
         <material name="blue"/>
@@ -214,5 +214,5 @@
         <visual>
         <geometry>
-            <mesh filename="file:///home/logicbomb/Projects/SLAM/wheely-dan/src/wd_description/meshes/wheel_right_link.stl" scale="0.001 0.001 0.001"/>
+            <mesh filename="$(find wd_description)/meshes/wheel_right_link.stl" scale="0.001 0.001 0.001"/>
         </geometry>
         <material name="blue"/>
@@ -243,5 +243,5 @@
         <visual>
         <geometry>
-            <mesh filename="file:///home/logicbomb/Projects/SLAM/wheely-dan/src/wd_description/meshes/caster_fork_link.stl" scale="0.001 0.001 0.001"/>
+            <mesh filename="$(find wd_description)/meshes/caster_fork_link.stl" scale="0.001 0.001 0.001"/>
         </geometry>
         <material name="dark_grey"/>
@@ -264,5 +264,5 @@
         <visual>
         <geometry>
-            <mesh filename="file:///home/logicbomb/Projects/SLAM/wheely-dan/src/wd_description/meshes/caster_wheel_link.stl" scale="0.001 0.001 0.001"/>
+            <mesh filename="$(find wd_description)/meshes/caster_wheel_link.stl" scale="0.001 0.001 0.001"/>
         </geometry>
         <material name="dark_grey"/>
@@ -292,5 +292,5 @@
         <visual>
         <geometry>
-            <mesh filename="file:///home/logicbomb/Projects/SLAM/wheely-dan/src/wd_description/meshes/caster_fork_link.stl" scale="0.001 0.001 0.001"/>
+            <mesh filename="$(find wd_description)/meshes/caster_fork_link.stl" scale="0.001 0.001 0.001"/>
         </geometry>
         <material name="dark_grey"/>
@@ -313,5 +313,5 @@
         <visual>
         <geometry>
-            <mesh filename="file:///home/logicbomb/Projects/SLAM/wheely-dan/src/wd_description/meshes/caster_wheel_link.stl" scale="0.001 0.001 0.001"/>
+            <mesh filename="$(find wd_description)/meshes/caster_wheel_link.stl" scale="0.001 0.001 0.001"/>
         </geometry>
         <material name="dark_grey"/>
@@ -342,5 +342,5 @@
         <origin xyz="0 0 0" rpy="${-pi/2} 0 ${-pi/2}"/>
         <geometry>
-            <mesh filename="file:///home/logicbomb/Projects/SLAM/wheely-dan/src/wd_description/meshes/d435.dae"/>
+            <mesh filename="$(find wd_description)/meshes/d435.dae"/>
         </geometry>
         <material name="dark_grey"/>
