Commit message: Rearrange xacro files

File: src/wd_description/urdf/robot_desc.xacro (robot description, xacro)
@@ -30,5 +30,5 @@
         <visual>
         <geometry>
-            <mesh filename="$(find wd_description)/meshes/chassis_link.stl" scale="0.001 0.001 0.001"/>
+            <mesh filename="package://wd_description/meshes/chassis_link.stl" scale="0.001 0.001 0.001"/>
         </geometry>
         <material name="grey"/>
@@ -53,5 +53,5 @@
         <visual>
         <geometry>
-            <mesh filename="$(find wd_description)/meshes/jetson_link.stl" scale="0.001 0.001 0.001"/>
+            <mesh filename="package://wd_description/meshes/jetson_link.stl" scale="0.001 0.001 0.001"/>
         </geometry>
         <material name="dark_grey"/>
@@ -75,5 +75,5 @@
         <visual>
         <geometry>
-            <mesh filename="$(find wd_description)/meshes/battery_link.stl" scale="0.001 0.001 0.001"/>
+            <mesh filename="package://wd_description/meshes/battery_link.stl" scale="0.001 0.001 0.001"/>
         </geometry>
         <material name="red"/>
@@ -97,5 +97,5 @@
         <visual>
         <geometry>
-            <mesh filename="$(find wd_description)/meshes/pcb_link.stl" scale="0.001 0.001 0.001"/>
+            <mesh filename="package://wd_description/meshes/pcb_link.stl" scale="0.001 0.001 0.001"/>
         </geometry>
         <material name="green"/>
@@ -119,5 +119,5 @@
         <visual>
         <geometry>
-            <mesh filename="$(find wd_description)/meshes/driver_left_link.stl" scale="0.001 0.001 0.001"/>
+            <mesh filename="package://wd_description/meshes/driver_left_link.stl" scale="0.001 0.001 0.001"/>
         </geometry>
         <material name="grey"/>
@@ -141,5 +141,5 @@
         <visual>
         <geometry>
-            <mesh filename="$(find wd_description)/meshes/driver_right_link.stl" scale="0.001 0.001 0.001"/>
+            <mesh filename="package://wd_description/meshes/driver_right_link.stl" scale="0.001 0.001 0.001"/>
         </geometry>
         <material name="grey"/>
@@ -163,5 +163,5 @@
         <visual>
         <geometry>
-            <mesh filename="$(find wd_description)/meshes/lidar_link.stl" scale="0.001 0.001 0.001"/>
+            <mesh filename="package://wd_description/meshes/lidar_link.stl" scale="0.001 0.001 0.001"/>
         </geometry>
         <material name="dark_grey"/>
@@ -185,5 +185,5 @@
         <visual>
         <geometry>
-            <mesh filename="$(find wd_description)/meshes/wheel_left_link.stl" scale="0.001 0.001 0.001"/>
+            <mesh filename="package://wd_description/meshes/wheel_left_link.stl" scale="0.001 0.001 0.001"/>
         </geometry>
         <material name="blue"/>
@@ -214,5 +214,5 @@
         <visual>
         <geometry>
-            <mesh filename="$(find wd_description)/meshes/wheel_right_link.stl" scale="0.001 0.001 0.001"/>
+            <mesh filename="package://wd_description/meshes/wheel_right_link.stl" scale="0.001 0.001 0.001"/>
         </geometry>
         <material name="blue"/>
@@ -243,5 +243,5 @@
         <visual>
         <geometry>
-            <mesh filename="$(find wd_description)/meshes/caster_fork_link.stl" scale="0.001 0.001 0.001"/>
+            <mesh filename="package://wd_description/meshes/caster_fork_link.stl" scale="0.001 0.001 0.001"/>
         </geometry>
         <material name="dark_grey"/>
@@ -264,5 +264,5 @@
         <visual>
         <geometry>
-            <mesh filename="$(find wd_description)/meshes/caster_wheel_link.stl" scale="0.001 0.001 0.001"/>
+            <mesh filename="package://wd_description/meshes/caster_wheel_link.stl" scale="0.001 0.001 0.001"/>
         </geometry>
         <material name="dark_grey"/>
@@ -292,5 +292,5 @@
         <visual>
         <geometry>
-            <mesh filename="$(find wd_description)/meshes/caster_fork_link.stl" scale="0.001 0.001 0.001"/>
+            <mesh filename="package://wd_description/meshes/caster_fork_link.stl" scale="0.001 0.001 0.001"/>
         </geometry>
         <material name="dark_grey"/>
@@ -313,5 +313,5 @@
         <visual>
         <geometry>
-            <mesh filename="$(find wd_description)/meshes/caster_wheel_link.stl" scale="0.001 0.001 0.001"/>
+            <mesh filename="package://wd_description/meshes/caster_wheel_link.stl" scale="0.001 0.001 0.001"/>
         </geometry>
         <material name="dark_grey"/>
@@ -342,5 +342,5 @@
         <origin xyz="0 0 0" rpy="${-pi/2} 0 ${-pi/2}"/>
         <geometry>
-            <mesh filename="$(find wd_description)/meshes/d435.dae"/>
+            <mesh filename="package://wd_description/meshes/d435.dae"/>
         </geometry>
         <material name="dark_grey"/>

File: src/wd_simulation/urdf/sim_robot.urdf.xacro (robot description, xacro)
@@ -2,12 +2,12 @@
 <robot xmlns:xacro="http://www.ros.org/wiki/xacro"  name="robot">
     <xacro:arg name="use_ros2_control" default="true"/>
-    <xacro:include filename="robot_desc.xacro" />
+    <xacro:include filename="package://wd_description/urdf/robot_desc.xacro" />
     <!-- Switch between ros2_control and Gazebo integrated diff-drive control -->
     <xacro:if value="$(arg use_ros2_control)">
-        <xacro:include filename="$(find wd_control)/urdf/ros2_control.xacro"/>
+        <xacro:include filename="package://wd_control/urdf/ros2_control.xacro"/>
     </xacro:if>
     <xacro:unless value="$(arg use_ros2_control)">
-        <xacro:include filename="$(find wd_simulation)/urdf/gazebo_control.xacro"/>
+        <xacro:include filename="package://wd_simulation/urdf/gazebo_control.xacro"/>
     </xacro:unless>
-    <xacro:include filename="$(find wd_simulation)/urdf/sensors.xacro"/>
+    <xacro:include filename="package://wd_simulation/urdf/sensors.xacro"/>
 </robot>

Commit message: Change naming of camera links

File: src/wd_description/urdf/robot_desc.xacro (robot description, xacro)
@@ -338,5 +338,5 @@
     </joint>
     <!-- ========= DEPTH CAMERA ========= -->
-    <link name="depth_camera_link">
+    <link name="camera_link">
         <visual>
         <origin xyz="0 0 0" rpy="${-pi/2} 0 ${-pi/2}"/>
@@ -353,17 +353,17 @@
         </inertial>
     </link>
-    <joint name="depth_camera_joint" type="fixed">
-        <parent link="base_link"/>
-        <child link="depth_camera_link"/>
+    <joint name="camera_joint" type="fixed">
+        <parent link="base_link"/>
+        <child link="camera_link"/>
         <origin xyz="0.2 0 0.075" rpy="0 0 0"/>
     </joint>
     <!-- ── Optical frame (ROS convention: z-forward, x-right, y-down) ── -->
-    <joint name="depth_camera_optical_joint" type="fixed">
-      <parent link="depth_camera_link"/>
-      <child  link="depth_camera_link_optical"/>
+    <joint name="camera_optical_joint" type="fixed">
+      <parent link="camera_link"/>
+      <child  link="camera_link_optical"/>
       <!-- Rotate from Gazebo (x-forward) to ROS optical (z-forward) convention -->
       <origin xyz="0 0 0" rpy="${-pi/2} 0 ${-pi/2}"/>
     </joint>
-    <link name="depth_camera_link_optical"/>
+    <link name="camera_link_optical"/>
     <!-- ========= GAZEBO SETTINGS ========= -->
     <gazebo reference="caster_wheel_left_link">

File: src/wd_simulation/urdf/sensors.xacro (robot description, xacro)
@@ -30,5 +30,5 @@
         </sensor>
     </gazebo>
-    <gazebo reference="depth_camera_link">
+    <gazebo reference="camera_link">
       <!-- Based on Intel realsense D435 (intrinsics and distortion not modeled)-->
       <sensor name="rs_front" type="rgbd_camera">
@@ -81,5 +81,5 @@
         </camera>
         <topic>camera/depth</topic>
-        <gz_frame_id>depth_camera_link_optical</gz_frame_id>
+        <gz_frame_id>camera_link_optical</gz_frame_id>
       </sensor>
     </gazebo>
